Commit message: Fix ergocub config files

File: ergocub_moveit_config/config/ergocub.ros2_control.xacro (robot description, xacro)
@@ -269,5 +269,5 @@
             </joint>
         </ros2_control>
-        <ros2_control name="left_arm_torso_${name}" type="system">
+        <ros2_control name="right_arm_torso_${name}" type="system">
           <hardware>
               <plugin>robot_controller/RobotController</plugin>
@@ -296,50 +296,50 @@
             <state_interface name="velocity"/>
         </joint>
-          <joint name="l_shoulder_pitch">
+          <joint name="r_shoulder_pitch">
             <command_interface name="position"/>
             <state_interface name="position">
-              <param name="initial_value">${initial_positions['l_shoulder_pitch']}</param>
+              <param name="initial_value">${initial_positions['r_shoulder_pitch']}</param>
             </state_interface>
             <state_interface name="velocity"/>
           </joint>
-          <joint name="l_shoulder_roll">
-              <command_interface name="position"/>
-              <state_interface name="position">
-                <param name="initial_value">${initial_positions['l_shoulder_roll']}</param>
-              </state_interface>
-              <state_interface name="velocity"/>
-          </joint>
-          <joint name="l_shoulder_yaw">
-              <command_interface name="position"/>
-              <state_interface name="position">
-                <param name="initial_value">${initial_positions['l_shoulder_yaw']}</param>
-              </state_interface>
-              <state_interface name="velocity"/>
-          </joint>
-          <joint name="l_elbow">
-              <command_interface name="position"/>
-              <state_interface name="position">
-                <param name="initial_value">${initial_positions['l_elbow']}</param>
-              </state_interface>
-              <state_interface name="velocity"/>
-          </joint>
-          <joint name="l_wrist_yaw">
-              <command_interface name="position"/>
-              <state_interface name="position">
-                <param name="initial_value">${initial_positions['l_wrist_yaw']}</param>
-              </state_interface>
-              <state_interface name="velocity"/>
-          </joint>
-          <joint name="l_wrist_roll">
-              <command_interface name="position"/>
-              <state_interface name="position">
-                <param name="initial_value">${initial_positions['l_wrist_roll']}</param>
-              </state_interface>
-              <state_interface name="velocity"/>
-          </joint>
-          <joint name="l_wrist_pitch">
-              <command_interface name="position"/>
-              <state_interface name="position">
-                <param name="initial_value">${initial_positions['l_wrist_pitch']}</param>
+          <joint name="r_shoulder_roll">
+              <command_interface name="position"/>
+              <state_interface name="position">
+                <param name="initial_value">${initial_positions['r_shoulder_roll']}</param>
+              </state_interface>
+              <state_interface name="velocity"/>
+          </joint>
+          <joint name="r_shoulder_yaw">
+              <command_interface name="position"/>
+              <state_interface name="position">
+                <param name="initial_value">${initial_positions['r_shoulder_yaw']}</param>
+              </state_interface>
+              <state_interface name="velocity"/>
+          </joint>
+          <joint name="r_elbow">
+              <command_interface name="position"/>
+              <state_interface name="position">
+                <param name="initial_value">${initial_positions['r_elbow']}</param>
+              </state_interface>
+              <state_interface name="velocity"/>
+          </joint>
+          <joint name="r_wrist_yaw">
+              <command_interface name="position"/>
+              <state_interface name="position">
+                <param name="initial_value">${initial_positions['r_wrist_yaw']}</param>
+              </state_interface>
+              <state_interface name="velocity"/>
+          </joint>
+          <joint name="r_wrist_roll">
+              <command_interface name="position"/>
+              <state_interface name="position">
+                <param name="initial_value">${initial_positions['r_wrist_roll']}</param>
+              </state_interface>
+              <state_interface name="velocity"/>
+          </joint>
+          <joint name="r_wrist_pitch">
+              <command_interface name="position"/>
+              <state_interface name="position">
+                <param name="initial_value">${initial_positions['r_wrist_pitch']}</param>
               </state_interface>
               <state_interface name="velocity"/>
